Commit message: hw2

File: assignments/staples/scara.urdf (robot description, URDF)
Before this commit: robot scara_robot, 5 links, 4 joints
Joints:
- joint link1_to_link2: origin xyz=0.92 0.0 0.08 rpy=0.0 0.0 0.0 -> xyz=0.90 0.0 0.08 rpy=0.0 0.0 0.0
- joint link2_to_plunger: axis 0.0 0.0 -1.0 -> 0.0 0.0 1.0; limit lower=-0.25 upper=0.0 effort=50.0 velocity=0.5 -> lower=-0.01 upper=0.24 effort=50.0 velocity=0.5; origin xyz=1.025 0.0 0.08 rpy=0.0 0.0 0.0 -> xyz=1.02 0.0 0.08 rpy=0.0 0.0 0.0
- joint plunger_to_ee: origin xyz=0.0 0.0 -0.46 rpy=0.0 0.0 0.0 -> xyz=0.0 0.0 -0.45 rpy=0.0 0.0 0.0
